Commit message: [bugfix] Fix typo intertial -> inertial + add dummy inertia

File: urdf/hoap3.urdf (robot description, URDF)
Before this commit: robot hoap3, 36 links, 35 joints
Links:
- link CHEST: mass None -> 3.26
- link H_PAN: mass None -> 7.10e-02
- link H_ROLL: mass None -> 4.12e-01
- link H_TILT: mass None -> 0
- link L_AAA: mass None -> 1.54e-01
- link L_AFE: mass None -> 1.95e-01
- link L_EB: mass None -> 2.16e-01
- link L_KN: mass None -> 3.28e-01
- link L_LAA: mass None -> 2.10e-01
- link L_LFE: mass None -> 5.19e-01
- link L_LR: mass None -> 5.87e-02
- link L_SAA: mass None -> 2.34e-01
- link L_SFE: mass None -> 2.10e-01
- link L_SHR: mass None -> 1.965e-01
- link R_AAA: mass None -> 1.54e-01
- link R_AFE: mass None -> 1.95e-01
- link R_EB: mass None -> 2.16e-01
- link R_KN: mass None -> 3.28e-01
- link R_LAA: mass None -> 2.10e-01
- link R_LFE: mass None -> 5.19e-01
- link R_LR: mass None -> 5.87e-02
- link R_SAA: mass None -> 2.34e-01
- link R_SFE: mass None -> 2.10e-01
- link R_SHR: mass None -> 1.965e-01
- link WAIST: mass None -> 4.17e-01
